File: Squama_Ethernet/Squama_Ethernet.sch (EAGLE design)
At the start: 62 parts, among them J1 HY931147C, J10 320110033, J11 320110033, U1 W5500, U3 CJ1117-3.3, U8 ATSAMD21, X1 32.768k, X2 25MHz

Commit message: add datasheet
Other:
- note removed: "Bruce"
- note removed: "Wangcf"
- note removed: "v1.0"
Changed lines of the file:
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@@
 <sheet>
 <plain>
-<text x="190.5" y="11.43" size="1.778" layer="97" ratio="10">Wangcf</text>
-<text x="223.52" y="11.43" size="1.778" layer="97" ratio="10">Bruce</text>
-<text x="223.52" y="5.08" size="1.778" layer="97" ratio="10">v1.0</text>
 </plain>
 <instances>
@@
 <sheet>
 <plain>
-<text x="184.15" y="11.43" size="1.778" layer="97" ratio="10">Wangcf</text>
-<text x="217.17" y="11.43" size="1.778" layer="97" ratio="10">Bruce</text>
-<text x="217.17" y="5.08" size="1.778" layer="97" ratio="10">v1.0</text>
 </plain>
 <instances>
